File: ENNOID_BMS/Slave/cell.kicad_sch (KiCad schematic)
At the start: 6 parts, among them Q16 TSM2323

Commit message: ENNOID BMS PCBs completed
Parts:
- Q16: footprint TO_SOT_Packages_SMD:SOT-23 -> Package_TO_SOT_SMD:SOT-23
Changed lines of the file:
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@@
 			)
 		)
-		(property "Footprint" "TO_SOT_Packages_SMD:SOT-23"
+		(property "Footprint" "Package_TO_SOT_SMD:SOT-23"
 			(at 83.82 106.68 0)
 			(effects
