File: ENNOID_BMS/Slave/LTC6812-15W.kicad_pcb (KiCad board)
At the start: 2 copper layers, 60 x 100 mm, 201 parts, among them J1 PB MB 2, J10 PB MB 1, J11 PA MA 1, J2 PA MA 2, J3 Sensors, J5 Cells, J6 Sensors, Q1 DZTT5551, Q10 TSM2323, Q11 TSM2323, Q12 TSM2323, Q13 TSM2323, Q14 TSM2323, Q15 TSM2323, Q16 TSM2323, Q17 DZTT5551, Q2 TSM2323, Q3 TSM2323, Q4 TSM2323, Q5 TSM2323, Q6 TSM2323, Q7 TSM2323, Q8 TSM2323, Q9 TSM2323, U1 LTC6812, U2 LTC6812

Commit message: slave pcb complete
Parts:
- removed C34: 100n, Capacitor_SMD:C_0603_1608Metric
- removed R68: 100k, Resistor_SMD:R_0603_1608Metric
- removed R97: 100, Resistor_SMD:R_0603_1608Metric
- removed TH1: 100k, Resistor_SMD:R_0805_2012Metric
- F10, F11, F12, F13, F14, F15, F16, F17, F18, F19, F4, F5, F6, F7, F8, F9: footprint ENNOID:FUSE -> Fuse:Fuse_0603_1608Metric
- moved J6 159.2 mm to (91.6, 120.5)
- moved Q17 152.8 mm to (67.2, 63.9), turned to -90 degrees
- moved J3 135.7 mm to (102.5, 68.5), turned to 0 degrees
- moved J2 117.7 mm to (104.7, 51.8), turned to 0 degrees
- moved C28 109.7 mm to (61.9, 67.1), turned to 0 degrees
- moved R11 109.6 mm to (60.7, 105.4)
- moved TR2 109.1 mm to (89.2, 65.3), turned to 0 degrees
- moved R82 107.0 mm to (86.0, 74.3), turned to 0 degrees
- moved R16 106.9 mm to (67.8, 105.3)
- moved C33 106.7 mm to (84.8, 76.2), turned to 0 degrees
- moved C26 106.3 mm to (69.1, 77.2), turned to -90 degrees
- moved C27 106.0 mm to (67.2, 77.2), turned to -90 degrees
- moved FB2 105.8 mm to (65.7, 73.9)
- moved R12 105.5 mm to (64.3, 105.3)
- moved J1 105.5 mm to (104.7, 60.5), turned to 0 degrees
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Connections:
- J3 pad 1: Meas8+ -> Meas15+
- J3 pad 10: Cell_12+ -> Cell_10+
- J3 pad 11: Meas13+ -> Meas10+
- J3 pad 12: Cell_13+ -> Cell_9+
- J3 pad 13: Meas14+ -> Meas9+
- J3 pad 14: Cell_14+ -> Cell_8+
- J3 pad 15: Meas15+ -> Meas8+
- J3 pad 2: Cell_8+ -> Cell_14+
- J3 pad 3: Meas9+ -> Meas14+
- J3 pad 4: Cell_9+ -> Cell_13+
- J3 pad 5: Meas10+ -> Meas13+
- J3 pad 6: Cell_10+ -> Cell_12+
- J3 pad 7: Meas11+ -> Meas12+
- J3 pad 9: Meas12+ -> Meas11+
- J6 pad 1: Cell_1- -> Cell_7+
- J6 pad 10: Meas5+ -> Meas3+
- J6 pad 11: Cell_5+ -> Cell_2+
- J6 pad 12: Meas6+ -> Meas2+
- J6 pad 13: Cell_6+ -> Cell_1+
- J6 pad 14: Meas7+ -> Meas1+
- J6 pad 15: Cell_7+ -> Cell_1-
- J6 pad 2: Meas1+ -> Meas7+
- J6 pad 3: Cell_1+ -> Cell_6+
- J6 pad 4: Meas2+ -> Meas6+
- J6 pad 5: Cell_2+ -> Cell_5+
- J6 pad 6: Meas3+ -> Meas5+
- J6 pad 7: Cell_3+ -> Cell_4+
- J6 pad 9: Cell_4+ -> Cell_3+
- U2 pad 38: Net-(U2-C0) -> Cell_1-
Routing:
- net Cell_1-: track 0.00 -> 160.1 mm, vias 0 -> 34
- net Cell_9+: track 0.00 -> 139.0 mm, vias 0 -> 2
- net Cell_8+: track 0.00 -> 135.6 mm, vias 0 -> 2
- net Cell_7+: track 0.00 -> 111.4 mm, vias 0 -> 2
- net Cell_15+: track 0.00 -> 102.7 mm, vias 0 -> 3
- net Net-(C4-Pad2): track 0.00 -> 100.7 mm, vias 0 -> 2
- net Cell_6+: track 0.00 -> 99.6 mm, vias 0 -> 2
- net Cell_10+: track 0.00 -> 93.3 mm, vias 0 -> 1
- net Cell_12+: track 0.00 -> 91.3 mm, vias 0 -> 2
- net Cell_11+: track 0.00 -> 90.1 mm, vias 0 -> 1
- net Cell_13+: track 0.00 -> 88.2 mm, vias 0 -> 2
- net Cell_14+: track 0.00 -> 88.2 mm, vias 0 -> 2
- net Cell_5+: track 0.00 -> 88.2 mm, vias 0 -> 2
- net /Vreg_2: track 0.00 -> 75.7 mm
- net Net-(D20-K): track 0.00 -> 74.2 mm
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- added copper zone on B.Cu, net Cell_1-
- added copper zone on F.Cu, net Cell_1-
Other:
- board size 60 x 100 mm -> 63.6 x 91.2 mm
