File: ENNOID_BMS/Slave/LTC6812-15W.kicad_sch (KiCad schematic)
At the start: 108 parts, among them J1 PB MB 2, J10 PB MB 1, J11 PA MA 1, J2 PA MA 2, J3 Sensors, J5 Cells, J6 Sensors, Q1 DZTT5551, Q17 DZTT5551, U1 LTC6812, U2 LTC6812

Commit message: precharge and discharge fixed
Other:
- note added: "HV"
- note added: "LV"
- note removed: "Meas- must be tied to its cell's negative. it is electrically isolated so this must be done This can either be done at the cells, or routed here and sent back, but this adds an additional 18 input wires"
Changed lines of the file:
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@@
 		(company "ENNOID")
+	)
+	(text "HV"
+		(exclude_from_sim no)
+		(at 875.03 158.75 0)
+		(effects
+			(font
+				(size 2.54 2.54)
+			)
+		)
 	)
 	(text "Cell Voltage and Balancing - Ennoid Slave with Thermistor GPIO inputs removed"
@@
 		)
 	)
-	(text "Meas- must be tied to its cell's negative. it is electrically isolated so this must be done\nThis can either be done at the cells, or routed here and sent back, but this adds an additional 18 input wires"
+	(text "LV"
 		(exclude_from_sim no)
-		(at 738.378 281.686 0)
+		(at 449.326 89.408 0)
 		(effects
 			(font
-				(size 1.27 1.27)
+				(size 2.54 2.54)
 			)
 		)
+	)
+	(text "LV"
+		(exclude_from_sim no)
+		(at 932.18 161.036 0)
+		(effects
+			(font
+				(size 2.54 2.54)
+			)
+		)
+	)
+	(text "HV"
+		(exclude_from_sim no)
+		(at 392.176 87.122 0)
+		(effects
+			(font
+				(size 2.54 2.54)
+			)
+		)

Commit message: Voltage measurement completed
Parts:
- added C34: 100n, Capacitor_SMD:C_0603_1608Metric, symbol Device:C
- added R68: 100k, Resistor_SMD:R_0603_1608Metric, symbol Device:R
- added TH1: 100k, Resistor_SMD:R_0805_2012Metric, symbol Device:Thermistor
Connections:
- net GND: now also C34.2, TH1.2
- net T1: now reaches U1.39 (GPIO1)
- net T1: now also C34.1, R68.2, TH1.1
- new net Vref2: R68.1
Other:
- note added: "Cell Voltage, Balancing, and Thermistor readings - Existing Ennoid Slave"
- note added: "Cell+ tap through bias resistor to Meas+ pin"
- note added: "Existing NTC Divider network to GPIO reading"
- note added: "IsoSPI transformer link"
- note added: "Per Cell stack configuration for Temperature measurement"
- note added: "Tie Meas- to Cell-"
- note removed: "Cell Voltage and Balancing - Ennoid Slave with Thermistor GPIO inputs removed"
- moved on the sheet: D4, J6, R10

Commit message: ENNOID BMS PCBs completed
Parts:
- J3, J6: footprint (none) -> Connector_PinHeader_2.54mm:PinHeader_1x15_P2.54mm_Horizontal
- J5: footprint Pin_Headers:Pin_Header_Angled_1x16_Pitch2.54mm -> Connector_PinHeader_2.54mm:PinHeader_1x16_P2.54mm_Horizontal
- Q1, Q17: footprint TO_SOT_Packages_SMD:SOT-223 -> Package_TO_SOT_SMD:SOT-223
- R11, R12, R16, R20, R24, R28, R32, R36, R40, R44, R48, R52, R56, R60, R64: footprint (none) -> Resistor_SMD:R_0603_1608Metric
Connections:
- net Vref2 is gone; now on net Vref2_1: R68.1
Changed lines of the file:
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@@
 		)
 	)
-	(label "Vref2"
+	(label "Vref2_1"
 		(at 358.14 177.8 180)
 		(effects
@@
 			)
 		)
-		(property "Footprint" "TO_SOT_Packages_SMD:SOT-223"
+		(property "Footprint" "Package_TO_SOT_SMD:SOT-223"
 			(at 314.96 101.6 0)
 			(effects
@@
 			)
 		)
-		(property "Footprint" "Pin_Headers:Pin_Header_Angled_1x16_Pitch2.54mm"
+		(property "Footprint" "Connector_PinHeader_2.54mm:PinHeader_1x16_P2.54mm_Horizontal"
 			(at 67.31 172.72 0)
 			(effects
@@
 			)
 		)
-		(property "Footprint" ""
+		(property "Footprint" "Resistor_SMD:R_0603_1608Metric"
 			(at 803.402 312.42 90)
 			(effects
@@
 			)
 		)
-		(property "Footprint" ""
+		(property "Footprint" "Resistor_SMD:R_0603_1608Metric"
 			(at 778.002 312.42 90)
 			(effects
@@
 			)
 		)
-		(property "Footprint" ""
+		(property "Footprint" "Resistor_SMD:R_0603_1608Metric"
 			(at 776.732 355.6 90)
 			(effects
@@
 			)
 		)
-		(property "Footprint" ""
+		(property "Footprint" "Resistor_SMD:R_0603_1608Metric"
 			(at 802.132 334.01 90)
 			(effects
@@
 			)
 		)
-		(property "Footprint" ""
+		(property "Footprint" "Resistor_SMD:R_0603_1608Metric"
 			(at 753.872 334.01 90)
 			(effects
@@
 			)
 		)
-		(property "Footprint" ""
+		(property "Footprint" "Resistor_SMD:R_0603_1608Metric"
 			(at 729.742 312.42 90)
 			(effects
@@
 			)
 		)
-		(property "Footprint" "TO_SOT_Packages_SMD:SOT-223"
+		(property "Footprint" "Package_TO_SOT_SMD:SOT-223"
 			(at 802.64 119.38 0)
 			(effects
@@
 			)
 		)
-		(property "Footprint" ""
+		(property "Footprint" "Resistor_SMD:R_0603_1608Metric"
 			(at 827.532 334.01 90)
 			(effects
@@
 			)
 		)
-		(property "Footprint" ""
+		(property "Footprint" "Resistor_SMD:R_0603_1608Metric"
 			(at 827.532 355.6 90)
 			(effects
@@
 			)
 		)
-		(property "Footprint" ""
+		(property "Footprint" "Connector_PinHeader_2.54mm:PinHeader_1x15_P2.54mm_Horizontal"
 			(at 621.03 255.27 0)
 			(effects
@@
 			)
 		)
-		(property "Footprint" ""
+		(property "Footprint" "Resistor_SMD:R_0603_1608Metric"
 			(at 729.742 334.01 90)
 			(effects
@@
 			)
 		)
-		(property "Footprint" ""
+		(property "Footprint" "Resistor_SMD:R_0603_1608Metric"
 			(at 753.872 312.42 90)
 			(effects
@@
 			)
 		)
-		(property "Footprint" ""
+		(property "Footprint" "Resistor_SMD:R_0603_1608Metric"
 			(at 778.002 334.01 90)
 			(effects
@@
 			)
 		)
-		(property "Footprint" ""
+		(property "Footprint" "Resistor_SMD:R_0603_1608Metric"
 			(at 753.872 354.33 90)
 			(effects
@@
 			)
 		)
-		(property "Footprint" ""
+		(property "Footprint" "Connector_PinHeader_2.54mm:PinHeader_1x15_P2.54mm_Horizontal"
 			(at 621.03 321.31 0)
 			(effects
@@
 			)
 		)
-		(property "Footprint" ""
+		(property "Footprint" "Resistor_SMD:R_0603_1608Metric"
 			(at 729.742 354.33 90)
 			(effects
@@
 			)
 		)
-		(property "Footprint" ""
+		(property "Footprint" "Resistor_SMD:R_0603_1608Metric"
 			(at 827.532 312.42 90)
 			(effects
@@
 			)
 		)
-		(property "Footprint" ""
+		(property "Footprint" "Resistor_SMD:R_0603_1608Metric"
 			(at 802.132 355.6 90)
 			(effects

Commit message: slave pcb complete
Parts:
- removed C34: 100n, Capacitor_SMD:C_0603_1608Metric, symbol Device:C
- removed R68: 100k, Resistor_SMD:R_0603_1608Metric, symbol Device:R
- removed R97: 100, Resistor_SMD:R_0603_1608Metric, symbol Device:R
- removed TH1: 100k, Resistor_SMD:R_0805_2012Metric, symbol Device:Thermistor
- F10, F11, F12, F13, F14, F15, F16, F17, F18, F19, F4, F5, F6, F7, F8, F9: footprint ENNOID:FUSE -> Fuse:Fuse_0603_1608Metric
Connections:
- net Cell_1+: now also J6.13 (Pin_13); no longer J6.3 (Pin_3)
- net Cell_10+: now also J3.10 (Pin_10); no longer J3.6 (Pin_6)
- net Cell_12+: now also J3.6 (Pin_6); no longer J3.10 (Pin_10)
- net Cell_13+: now also J3.4 (Pin_4); no longer J3.12 (Pin_12)
- net Cell_14+: now also J3.2 (Pin_2); no longer J3.14 (Pin_14)
- net Cell_2+: now also J6.11 (Pin_11); no longer J6.5 (Pin_5)
- net Cell_3+: now also J6.9 (Pin_9); no longer J6.7 (Pin_7)
- net Cell_4+: now also J6.7 (Pin_7); no longer J6.9 (Pin_9)
- net Cell_5+: now also J6.5 (Pin_5); no longer J6.11 (Pin_11)
- net Cell_6+: now also J6.3 (Pin_3); no longer J6.13 (Pin_13)
- net Cell_7+: now also J6.1 (Pin_1); no longer J6.15 (Pin_15)
- net Cell_8+: now also J3.14 (Pin_14); no longer J3.2 (Pin_2)
- net Cell_9+: now also J3.12 (Pin_12); no longer J3.4 (Pin_4)
- net GND: now also J6.15 (Pin_15), U2.38 (C0); no longer J6.1 (Pin_1)
- net Meas1+: now also J6.14 (Pin_14); no longer J6.2 (Pin_2)
- net Meas10+: now also J3.11 (Pin_11); no longer J3.5 (Pin_5)
- net Meas11+: now also J3.9 (Pin_9); no longer J3.7 (Pin_7)
- net Meas12+: now also J3.7 (Pin_7); no longer J3.9 (Pin_9)
- net Meas13+: now also J3.5 (Pin_5); no longer J3.11 (Pin_11)
- net Meas14+: now also J3.3 (Pin_3); no longer J3.13 (Pin_13)
- net Meas15+: now also J3.1 (Pin_1); no longer J3.15 (Pin_15)
- net Meas2+: now also J6.12 (Pin_12); no longer J6.4 (Pin_4)
- net Meas3+: now also J6.10 (Pin_10); no longer J6.6 (Pin_6)
- net Meas5+: now also J6.6 (Pin_6); no longer J6.10 (Pin_10)
- net Meas6+: now also J6.4 (Pin_4); no longer J6.12 (Pin_12)
- net Meas7+: now also J6.2 (Pin_2); no longer J6.14 (Pin_14)
- net Meas8+: now also J3.15 (Pin_15); no longer J3.1 (Pin_1)
- net Meas9+: now also J3.13 (Pin_13); no longer J3.3 (Pin_3)
Other:
- note removed: "Existing NTC Divider network to GPIO reading"
- moved on the sheet: J3, J6
