File: ENNOID_BMS/Slave/LTC6812-15W.kicad_sch (KiCad schematic)
At the start: 153 parts, among them J1 PB MB 2, J10 PB MB 1, J11 PA MA 1, J2 PA MA 2, J3 Sensors, J5 Cells, J6 Sensors, Q1 DZTT5551, Q17 DZTT5551, Q18 2N7002, Q19 2N7002, Q20 2N7002, Q21 2N7002, Q22 2N7002, Q23 2N7002, Q24 2N7002, Q25 2N7002, Q26 2N7002, Q27 2N7002, Q28 2N7002, Q29 2N7002, Q30 2N7002, Q31 2N7002, Q32 2N7002, U1 LTC6812-1, U2 LTC6812-1

Commit message: Slave with SMD and no other fuses
Parts:
- removed F10, F11, F12, F13, F14, F15, F16, F17, F18, F19, F4, F5, F6, F7, F8, F9: 0.25A, Fuse:Fuse_0603_1608Metric, symbol Device:Fuse
- removed J5: Cells, Connector_JST:JST_XH_S16B-XH-A_1x16_P2.50mm_Horizontal, symbol Connector_Generic:Conn_01x16
- added J4, J5: Conn_01x08, Connector_Molex:Molex_PicoBlade_53048-0810_1x08_P1.25mm_Horizontal, symbol Connector_Generic:Conn_01x08
- F1, F2, F20, F21, F22, F23, F24, F25, F26, F27, F28, F29, F3, F30, F31, F32: value Fuse -> 5A; Part Number (none) -> 0885005.DR
- J1, J10, J11, J2: footprint Connector_JST:JST_XH_B2B-XH-A_1x02_P2.50mm_Vertical -> Connector_Molex:Molex_PicoBlade_53048-0210_1x02_P1.25mm_Horizontal; Part Number B2B-XH-A -> 53048-0210
- J3, J6: footprint Connector_JST:JST_XH_S15B-XH-A_1x15_P2.50mm_Horizontal -> Connector_Molex:Molex_PicoBlade_53048-1510_1x15_P1.25mm_Horizontal; Part Number S15B-XH-A(LF)(SN) -> 53048-1510
- Q18, Q19, Q20, Q21, Q22, Q23, Q24, Q25, Q26, Q27, Q28, Q29, Q30, Q31, Q32: Part Number (none) -> 2N7002
- R11, R12, R16, R20, R24, R28, R32, R36, R40, R44, R48, R52, R56, R60, R64: Part Number CRCW0603680RFKEA -> ERJ-UP3F6800V
Connections:
- net Cell_1+: now also F31.2
- net Cell_10+: now also F22.2, J3.10 (Pin_10); no longer J3.6 (Pin_6)
- net Cell_11+: now also F21.2
- net Cell_12+: now also F20.2, J3.6 (Pin_6); no longer J3.10 (Pin_10)
- net Cell_13+: now also F3.2, J3.4 (Pin_4); no longer J3.12 (Pin_12)
- net Cell_14+: now also F2.2, J3.2 (Pin_2); no longer J3.14 (Pin_14)
- net Cell_15+: now also F1.2
- net Cell_2+: now also F30.2
- net Cell_3+: now also F29.2
- net Cell_4+: now also F28.2
- net Cell_5+: now also F27.2
- net Cell_6+: now also F26.2
- net Cell_7+: now also F25.2
- net Cell_8+: now also F24.2, J3.14 (Pin_14); no longer J3.2 (Pin_2)
- net Cell_9+: now also F23.2, J3.12 (Pin_12); no longer J3.4 (Pin_4)
- net GND: now also F32.2
- net ISO_1A_N: now also J10.2 (Pin_2); no longer J10.1 (Pin_1)
- net ISO_1A_P: now also J10.1 (Pin_1); no longer J10.2 (Pin_2)
- net ISO_1B_N: now also J11.2 (Pin_2); no longer J11.1 (Pin_1)
- net ISO_1B_P: now also J11.1 (Pin_1); no longer J11.2 (Pin_2)
- net ISO_2A_N: now also J2.1 (Pin_1); no longer J1.1 (Pin_1)
- net ISO_2A_P: now also J2.2 (Pin_2); no longer J1.2 (Pin_2)
- net ISO_2B_N: now also J1.1 (Pin_1); no longer J2.2 (Pin_2)
- net ISO_2B_P: now also J1.2 (Pin_2); no longer J2.1 (Pin_1)
- net Meas10+: now also J3.11 (Pin_11); no longer J3.5 (Pin_5)
- net Meas11+: now also J3.9 (Pin_9); no longer J3.7 (Pin_7)
- net Meas12+: now also J3.7 (Pin_7); no longer J3.9 (Pin_9)
- net Meas13+: now also J3.5 (Pin_5); no longer J3.11 (Pin_11)
- net Meas14+: now also J3.3 (Pin_3); no longer J3.13 (Pin_13)
- net Meas15+: now also J3.1 (Pin_1); no longer J3.15 (Pin_15)
- net Meas8+: now also J3.15 (Pin_15); no longer J3.1 (Pin_1)
- net Meas9+: now also J3.13 (Pin_13); no longer J3.3 (Pin_3)
- net at F20.1: now also J4.5 (Pin_5)
- net at F32.1: now also J5.1 (Pin_1)
- net at F1.1: now also J4.8 (Pin_8)
- net at F3.1: now also J4.6 (Pin_6)
- net at F28.1: now also J5.5 (Pin_5)
- net at F2.1: now also J4.7 (Pin_7)
- net at F21.1: now also J4.4 (Pin_4)
- net at F25.1: now also J5.8 (Pin_8)
- net at F30.1: now also J5.3 (Pin_3)
- net at F23.1: now also J4.2 (Pin_2)
- net at F31.1: now also J5.2 (Pin_2)
- net at F27.1: now also J5.6 (Pin_6)
- net at F26.1: now also J5.7 (Pin_7)
- net at F22.1: now also J4.3 (Pin_3)
- net at F24.1: now also J4.1 (Pin_1)
- net at F29.1: now also J5.4 (Pin_4)
- net T1: no longer names the net of U1.39 (GPIO1)
Other:
- note added: "Potential 1500A@125VDC fault fuses Little Fuse 0885005.DR"
- note removed: "Potential 1500A@125VDC fault fuses"
- moved on the sheet: D4, F1, J1, J2, J3, R10

Commit message: fused slave variant v1
Parts:
- removed F2, F20, F21, F22, F23, F24, F25, F26, F27, F28, F29, F3, F30, F31, F32: 5A, ENNOID:FUSC10948X488N, symbol Device:Fuse
- added F17, F18, F19, F35, F36, F37, F38, F39, F40, F41, F42, F43, F44, F45, F46, F47, F48, F49, F50, F51, F52, F53, F54, F55, F56, F57, F58, F59, F60, F61, F62, F63, F64, F65, F66, F67: 50mA, Fuse:Fuse_0603_1608Metric, symbol Device:Fuse
- F1: value 5A -> 50mA; footprint ENNOID:FUSC10948X488N -> Fuse:Fuse_0603_1608Metric; Part Number 0885005.DR -> F0603G0R05FNTR
Connections:
- net Cell_1+: now also J5.2 (Pin_2)
- net Cell_10+: now also J4.3 (Pin_3)
- net Cell_11+: now also J4.4 (Pin_4)
- net Cell_12+: now also J4.5 (Pin_5)
- net Cell_13+: now also J4.6 (Pin_6)
- net Cell_14+: now also J4.7 (Pin_7)
- net Cell_15+: now also J4.8 (Pin_8); no longer F1.2
- net Cell_2+: now also J5.3 (Pin_3)
- net Cell_3+: now also J5.4 (Pin_4)
- net Cell_4+: now also J5.5 (Pin_5)
- net Cell_5+: now also J5.6 (Pin_6)
- net Cell_6+: now also J5.7 (Pin_7)
- net Cell_7+: now also J5.8 (Pin_8)
- net Cell_8+: now also J4.1 (Pin_1)
- net Cell_9+: now also J4.2 (Pin_2)
- net GND: now also J5.1 (Pin_1), F19.1, F53.2, F65.2; no longer U1.65 (V-), U2.38 (C0), U2.65 (V-)
- net S1: now also F52.2; no longer U2.37 (S1)
- net S10: now also F17.2; no longer U2.17 (S10)
- net S11: now also F54.1; no longer U2.13 (S11)
- net S12: now also F56.1; no longer U2.11 (S12)
- net S13: now also F58.1; no longer U2.9 (S13)
- net S14: now also F60.1; no longer U2.7 (S14)
- net S15: now also F62.1; no longer U2.5 (S15)
- net S2: now also F50.2; no longer U2.35 (S2)
- net S3: now also F48.2; no longer U2.33 (S3)
- net S4: now also F45.2; no longer U2.31 (S4)
- net S5: now also F43.2; no longer U2.29 (S5)
- net S6: now also F42.2; no longer U2.25 (S6)
- net S7: now also F40.2; no longer U2.23 (S7)
- net S8: now also F38.2; no longer U2.21 (S8)
- net S9: now also F36.2; no longer U2.19 (S9)
- net Vreg_1: now also F18.2; no longer C5.2, C6.2, C7.2, Q1.3 (E)
- net Vreg_2: now also F66.1; no longer C29.2, C30.2, C31.2, Q17.3 (E)
- net at C1.2, R1.1: now also F1.1; no longer U1.1 (V+)
- net at R89.1: now also F64.1; no longer U2.16 (C10)
- net at C10.2, R74.1: now also F67.1; no longer U2.1 (V+)
- net at R96.1: now also F46.2; no longer U2.32 (C3)
- net at R95.1: now also F44.2; no longer U2.30 (C4)
- net at U2.28 (C5): now also F47.1; no longer R94.1
- net at R86.1: now also F59.1; no longer U2.8 (C13)
- net at U2.10 (C12): now also F57.2; no longer R87.1
- net at U2.12 (C11): now also F55.2; no longer R88.1
- net at U2.18 (C9): now also F35.1; no longer R90.1
- net at U2.20 (C8): now also F37.1; no longer R91.1
- net at U2.22 (C7): now also F39.1; no longer R92.1
- net at U2.24 (C6): now also F41.1; no longer R93.1
- net at U2.34 (C2): now also F49.1; no longer R99.2
- net at U2.36 (C1): now also F51.1; no longer R98.2
- net at U2.4 (C15): now also F63.2; no longer R84.1
- net at U2.6 (C14): now also F61.2; no longer R85.1
- new net: C5.2, C6.2, C7.2, F18.1, Q1.3 (E)
- new net: F1.2, U1.1 (V+)
- new net: F19.2, U1.65 (V-)
- new net: F45.1, U2.31 (S4)
- new net: F47.2, R94.1
- new net: F42.1, U2.25 (S6)
- new net: C29.2, C30.2, C31.2, F66.2, Q17.3 (E)
- new net: F37.2, R91.1
- new net: F58.2, U2.9 (S13)
- new net: F62.2, U2.5 (S15)
- new net: F38.1, U2.21 (S8)
- new net: F49.2, R99.2
- new net: F48.1, U2.33 (S3)
- new net: F67.2, U2.1 (V+)
- new net: F56.2, U2.11 (S12)
- new net: F54.2, U2.13 (S11)
- new net: F44.1, U2.30 (C4)
- new net: F35.2, R90.1
- new net: F46.1, U2.32 (C3)
- new net: F59.2, U2.8 (C13)
- new net: F64.2, U2.16 (C10)
- new net: F17.1, U2.17 (S10)
- new net: F36.1, U2.19 (S9)
- new net: F40.1, U2.23 (S7)
- new net: F43.1, U2.29 (S5)
- new net: F50.1, U2.35 (S2)
- new net: F52.1, U2.37 (S1)
- new net: F53.1, U2.38 (C0)
- new net: F65.1, U2.65 (V-)
- new net: F60.2, U2.7 (S14)
- new net: F63.1, R84.1
- new net: F57.1, R87.1
- new net: F55.1, R88.1
- new net: F61.1, R85.1
- new net: F41.2, R93.1
- new net: F39.2, R92.1
- new net: F51.2, R98.2
Other:
- note removed: "Potential 1500A@125VDC fault fuses Little Fuse 0885005.DR"
- moved on the sheet: R84, R85, R86, R87, R88, R89, R90, R91, R92, R93, R94, R95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

Commit message: fuse boards
Parts:
- removed F17, F36, F38, F40, F42, F43, F45, F48, F50, F52, F54, F56, F58, F60, F62: 50mA, Fuse:Fuse_0603_1608Metric, symbol Device:Fuse
- R1, R3, R74, R76, R8, R81, R82, R84, R85, R86, R87, R88, R89, R9, R90, R91, R92, R93, R94, R95, R96, R98, R99: Part Number CRCW0603100RFKEA -> RCS0603100RFKEA
- R100, R101, R102, R103, R104, R105, R106, R107, R108, R109, R110, R68, R72, R73, R97: footprint Resistor_SMD:R_0603_1608Metric -> Resistor_SMD:R_0508_1220Metric; Part Number CRCW06033K30FKEA -> WK73R2ATTD3301F
- R11, R12, R16, R20, R24, R28, R32, R36, R40, R44, R48, R52, R56, R60, R64: Part Number ERJ-UP3F6800V -> RCS0603680RFKEA
Connections:
- net S1: now also U2.37 (S1)
- net S10: now also U2.17 (S10)
- net S11: now also U2.13 (S11)
- net S12: now also U2.11 (S12)
- net S13: now also U2.9 (S13)
- net S14: now also U2.7 (S14)
- net S15: now also U2.5 (S15)
- net S2: now also U2.35 (S2)
- net S3: now also U2.33 (S3)
- net S4: now also U2.31 (S4)
- net S5: now also U2.29 (S5)
- net S6: now also U2.25 (S6)
- net S7: now also U2.23 (S7)
- net S8: now also U2.21 (S8)
- net S9: now also U2.19 (S9)

Commit message: master and slave updated
Parts:
- removed F19, F53, F65: 50mA, Fuse:Fuse_0603_1608Metric, symbol Device:Fuse
- F1, F18, F35, F37, F39, F41, F44, F46, F47, F49, F51, F55, F57, F59, F61, F63, F64, F66, F67: footprint Fuse:Fuse_0603_1608Metric -> Fuse:Fuse_1206_3216Metric; Part Number F0603G0R05FNTR -> 3413.0002.11
Connections:
- net GND: now also U1.65 (V-), U2.38 (C0), U2.65 (V-)
- net Vreg_1: now also C5.2, C6.2, C7.2, Q1.3 (E); no longer F18.2
- net Vreg_2: now also C29.2, C30.2, C31.2, Q17.3 (E); no longer F66.1
- net at F1.1, R1.1: no longer C1.2
- net at C4.2, Q1.2 (C), Q1.4 (C): now also F18.2; no longer R3.1
- net at F1.2, U1.1 (V+): now also C1.2
- net at F67.1, R74.1: no longer C10.2
- net at F67.2, U2.1 (V+): now also C10.2
- net at C28.2, Q17.2 (C), Q17.4 (C): now also F66.1; no longer R76.1
- new net: F18.1, R3.1
- new net: F66.2, R76.1
Other:
- note added: "C0 does not require a 50mA fuse, since there are no other components to protect"
- moved on the sheet: C1, C10, F1, F18, F66, F67, FB1, FB2, R1, R3, R74, R76

Commit message: new cells and updated slave
Parts:
- R1, R3, R74, R76, R8, R81, R82, R84, R85, R86, R87, R88, R89, R9, R90, R91, R92, R93, R94, R95, R96, R98, R99: footprint Resistor_SMD:R_0603_1608Metric -> Resistor_SMD:R_0805_2012Metric; Part Number RCS0603100RFKEA -> CRCW0805100RFKEAHP

Commit message: added author
Other:
- company: ENNOID -> UCD Formula Student
Changed lines of the file:
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@@
 		(title "BMS-Slave")
 		(rev "V0.1")
-		(company "ENNOID")
+		(company "UCD Formula Student")
 		(comment 1 "Author: Keelan Reilly")
 	)
