File: BSPD_KR/BSPD KiCAD.kicad_pcb (KiCad board)
At the start: 2 copper layers, 58 x 84.6 mm, 75 parts, among them J1 Conn_01x03, J2 Conn_01x02, J3 Conn_01x02, K1 G5Q-1A4-DC12, Q1 2N7000, Q2 2N7000, U1 LM741CN/NOPB, U18 SN74AHCT1G08DBVR, U19 LM339N, U2 LM741CN/NOPB, U3 LM741CN/NOPB, U4 LM7805MPX/NOPB, U5 LM339N, U6 SN74AHC1G02DBVR, U9 SN74LVC1G04DBVT

Commit message: Slave with SMD and no other fuses
Parts:
- removed C1, C2, C3: 0.1uF, FA14_Capacitor:FA18X7R1H104KNU00
- removed Q2: 2N7000, Package_TO_SOT_THT:TO-92_Inline
- removed the REF** at (87.5, 112.1)
- removed the REF** at (40.1, 38.6)
- removed the REF** at (39.9, 112.1)
- removed the REF** at (87.5, 38.8)
- removed U1, U2, U3: LM741CN/NOPB, Package_DIP:DIP-8_W7.62mm
- added G***: LOGO, LOGO, F.Cu at (-192.0, 47.8)
- added G***: LOGO, LOGO, F.Cu at (-186.8, 39.3)
- added Q3: 2N7002, Package_TO_SOT_SMD:SOT-23, F.Cu at (-157.6, 103.7)
- added REF**: MountingHole_3.2mm_M3, MountingHole:MountingHole_3.2mm_M3, F.Cu at (-151.8, 39.6)
- added REF**: MountingHole_3.2mm_M3, MountingHole:MountingHole_3.2mm_M3, F.Cu at (-194.1, 110.5)
- added REF**: MountingHole_3.2mm_M3, MountingHole:MountingHole_3.2mm_M3, F.Cu at (-151.3, 110.7)
- added REF**: MountingHole_3.2mm_M3, MountingHole:MountingHole_3.2mm_M3, F.Cu at (-194.1, 39.6)
- C12, C5, C6, C7, C8, C9: footprint FA14_Capacitor:FA18X7R1H104KNU00 -> Kicad_Libraries:FA18X7R1H104KNU00
- C4: footprint FA14_Capacitor:FA14X7R1H224KNU00 -> Kicad_Libraries:FA14X7R1H224KNU00
- LED1, LED2, LED3, LED4, LED5: footprint LTL1CHG:LTL1CHG -> Kicad_Libraries:LTL1CHG
- Q1: value 2N7000 -> 2N7002; footprint Package_TO_SOT_THT:TO-92_Inline -> Package_TO_SOT_SMD:SOT-23
- U19, U5: footprint LM339N:DIP794W53P254L1930H508Q14N -> Kicad_Libraries:DIP794W53P254L1930H508Q14N
- moved Q1 274.7 mm to (-185.4, 65.1), turned to -90 degrees
- moved J2 272.6 mm to (-184.6, 109.2), turned to 0 degrees
- moved R18 256.9 mm to (-171.0, 40.0), turned to 0 degrees
- moved C6 256.3 mm to (-163.4, 110.2), turned to 0 degrees
- moved LED3 254.1 mm to (-164.5, 45.5), turned to 90 degrees
- moved LED4 253.6 mm to (-163.9, 79.4), turned to 90 degrees
- moved LED5 253.3 mm to (-163.7, 71.6)
- moved TP3 251.7 mm to (-158.9, 48.8), turned to 90 degrees
- moved C11 250.6 mm to (-174.1, 108.7), turned to 180 degrees
- moved U9 249.6 mm to (-157.4, 109.5), turned to 90 degrees
- moved K1 248.7 mm to (-195.6, 83.5), turned to -90 degrees
- moved R19 247.4 mm to (-160.9, 103.3)
- moved R21 247.4 mm to (-160.8, 106.7)
- moved U4 246.7 mm to (-193.5, 58.7), turned to 180 degrees
- moved C5 246.0 mm to (-186.7, 55.0)
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Connections:
- J1 pad 1: BRAKE_SENSOR_REAR -> BRAKE_SENSOR_FRONT
- J1 pad 2: CURRENT_SENSOR -> BRAKE_SENSOR_REAR
- J1 pad 3: BRAKE_SENSOR_FRONT -> CURRENT_SENSOR
- J3 pad 1: GLV- -> GLV+
- J3 pad 2: GLV+ -> GLV-
- Q1 pad 1: Net-(Q1-S) -> Net-(Q1-G)
- Q1 pad 2: Net-(Q1-G) -> GLV-
- Q1 pad 3: +5V -> Net-(D9-A)
- R1 pad 2: CURRENT_SENSOR_{BUF} -> CURRENT_SENSOR
- R19 pad 1: Net-(Q1-S) -> Net-(Q3-S)
- R2 pad 2: BRAKE_SENSOR_FRONT_{BUF} -> BRAKE_SENSOR_FRONT
- R27 pad 2: Net-(Q2-G) -> Net-(Q1-G)
- R29 pad 2: Net-(Q2-G) -> Net-(Q1-G)
- R3 pad 2: BRAKE_SENSOR_REAR_{BUF} -> BRAKE_SENSOR_REAR
- R4 pad 2: CURRENT_SENSOR_{BUF} -> CURRENT_SENSOR
- R5 pad 2: BRAKE_SENSOR_FRONT_{BUF} -> BRAKE_SENSOR_FRONT
- R6 pad 2: BRAKE_SENSOR_REAR_{BUF} -> BRAKE_SENSOR_REAR
- U5 pad 14: Net-(Q2-G) -> Net-(Q1-G)
- U9 pad 4: Net-(Q1-G) -> Net-(Q3-G)
Routing:
- net GLV+: track 161.7 -> 76.7 mm
- net Net-(Q1-G): track 4.85 -> 53.7 mm
- net Net-(U18-Pad4): track 2.84 -> 38.1 mm
- net Net-(R15-Pad1): track 18.8 -> 44.3 mm, vias 0 -> 1
- net Net-(U5A-+): track 36.2 -> 15.3 mm
- net BRAKE_SENSOR_FRONT_{BUF}: track 19.6 -> 0.00 mm
- net CURRENT_SENSOR_{BUF}: track 18.7 -> 0.00 mm
- net Net-(R26-Pad1): track 27.5 -> 45.2 mm, vias 0 -> 1
- net Net-(Q2-G): track 16.6 -> 0.00 mm
- net Net-(U19A-+): track 30.5 -> 15.4 mm
- net BRAKE_SENSOR_REAR_{BUF}: track 14.8 -> 0.00 mm
- net /500ms: track 23.4 -> 9.10 mm
- net Net-(R14-Pad1): track 13.3 -> 27.2 mm
- net Net-(U19C--): track 29.3 -> 16.2 mm
- net Net-(U5A--): track 34.0 -> 21.1 mm
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Other:
- board size 58 x 84.6 mm -> 52.2 x 80.9 mm
