File: BSPD_KR/BSPD KiCAD.kicad_sch (KiCad schematic)
At the start: 65 parts, among them J1 Conn_01x03, J2 Conn_01x02, J3 Conn_01x02, K1 G5Q-1A4-DC12, Q1 2N7002, Q3 2N7002, U18 SN74AHCT1G08DBVR, U19 LM339N, U4 LM7805MPX/NOPB, U5 LM339N, U6 SN74AHC1G02DBVR, U9 SN74LVC1G04DBVT

Commit message: bspd comments
Other:
- note added: "Current sensor potentiometer should be set to whatever sensor outputs at 16A V_threshold = 2.5 V + (15.9 A × 0.010 V/A) ≈ 2.66 V or better: TP4 = zero-current sensor voltage + 0.16 V"
- note removed: "Should be set to whatever sensor outputs at 16A V_threshold = 2.5 V + (15.9 A × 0.010 V/A) ≈ 2.66 V or better: TP4 = zero-current sensor voltage + 0.16 V"
Changed lines of the file:
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@@
 		(comment 2 "Updated by: Keelan Reilly")
 	)
-	(text "Should be set to whatever sensor outputs at 16A\n\nV_threshold = 2.5 V + (15.9 A × 0.010 V/A) ≈ 2.66 V\n\nor better:\n\nTP4 = zero-current sensor voltage + 0.16 V\n\n"
+	(text "Current sensor potentiometer should be set to whatever sensor outputs at 16A\n\nV_threshold = 2.5 V + (15.9 A × 0.010 V/A) ≈ 2.66 V\n\nor better:\n\nTP4 = zero-current sensor voltage + 0.16 V\n\n"
 		(exclude_from_sim no)
-		(at 89.916 87.122 0)
+		(at 78.994 112.268 0)
 		(effects
 			(font
@@
 	(text "ALl LEDs are off when BSPD is OK"
 		(exclude_from_sim no)
-		(at 85.598 172.466 0)
+		(at 77.216 150.876 0)
 		(effects
 			(font
@@
 		)
 	)
-	(text "Anything below 0.455 volts is invalid\n20 bar corresponds 2.8V\n25 bar corresponds to 3.36V\n30 bar correspons to 3.93v"
+	(text "Anything below 0.455 volts is invalid\n\n20 bar corresponds 2.8V\n25 bar corresponds to 3.36V\n30 bar correspons to 3.93v"
 		(exclude_from_sim no)
-		(at 96.266 136.906 0)
+		(at 78.232 137.414 0)
 		(effects
 			(font
@@
 	(text "BSPD is closed when NOT( hard braking AND too much power for >500 ms )"
 		(exclude_from_sim no)
-		(at 79.756 106.172 0)
+		(at 78.486 125.984 0)
 		(effects
 			(font
