File: ENNOID_BMS/Cell Tap Fuse Board/Cell Tap Fuse Board.kicad_pcb (KiCad board)
At the start: 2 copper layers, 30 x 16 mm, 3 parts, among them J1 Conn_01x02

Commit message: master and slave updated
Parts:
- added F2: C308F-V-250MA-TR1, Kicad_Libraries:C308F-V-250MA-TR1, F.Cu at (81.3, 114.5)
- added F3: C308F-V-250MA-TR1, Kicad_Libraries:C308F-V-250MA-TR1, F.Cu at (94.7, 72.7)
- added F4: C308F-V-250MA-TR1, Kicad_Libraries:C308F-V-250MA-TR1, F.Cu at (81.3, 236.2)
- added F5: C308F-V-250MA-TR1, Kicad_Libraries:C308F-V-250MA-TR1, F.Cu at (81.3, 317.4)
- added F6: C308F-V-250MA-TR1, Kicad_Libraries:C308F-V-250MA-TR1, F.Cu at (81.3, 155.1)
- added F7: C308F-V-250MA-TR1, Kicad_Libraries:C308F-V-250MA-TR1, F.Cu at (81.1, 195.9)
- added F8: C308F-V-250MA-TR1, Kicad_Libraries:C308F-V-250MA-TR1, F.Cu at (81.6, 277.0)
- added G***: LOGO, LOGO, F.Cu at (89.2, 177.4)
- added G***: LOGO, LOGO, F.Cu at (89.0, 167.4)
- added H2: MountingHole_Pad, MountingHole:MountingHole_5.5mm_Pad, F.Cu at (76.0, 113.6)
- added H3: MountingHole_Pad, MountingHole:MountingHole_5.5mm_Pad, F.Cu at (76.0, 73.0)
- added H4: MountingHole_Pad, MountingHole:MountingHole_5.5mm_Pad, F.Cu at (76.0, 235.6)
- added H5: MountingHole_Pad, MountingHole:MountingHole_5.5mm_Pad, F.Cu at (76.0, 316.9)
- added H6: MountingHole_Pad, MountingHole:MountingHole_5.5mm_Pad, F.Cu at (76.0, 154.3)
- added H7: MountingHole_Pad, MountingHole:MountingHole_5.5mm_Pad, F.Cu at (76.0, 194.9)
- added H8: MountingHole_Pad, MountingHole:MountingHole_5.5mm_Pad, F.Cu at (76.0, 276.3)
- added J2: Conn_01x02, Connector_Molex:Molex_PicoBlade_53047-0210_1x02_P1.25mm_Vertical, F.Cu at (85.0, 103.1)
- added J3: Conn_01x02, Connector_Molex:Molex_PicoBlade_53047-0210_1x02_P1.25mm_Vertical, F.Cu at (85.1, 83.0)
- added J4: Conn_01x02, Connector_Molex:Molex_PicoBlade_53047-0210_1x02_P1.25mm_Vertical, F.Cu at (84.9, 225.1)
- added J5: Conn_01x02, Connector_Molex:Molex_PicoBlade_53047-0210_1x02_P1.25mm_Vertical, F.Cu at (85.6, 306.2)
- added J6: Conn_01x02, Connector_Molex:Molex_PicoBlade_53047-0210_1x02_P1.25mm_Vertical, F.Cu at (85.2, 143.8)
- added J7: Conn_01x02, Connector_Molex:Molex_PicoBlade_53047-0210_1x02_P1.25mm_Vertical, F.Cu at (85.4, 184.5)
- added J8: Conn_01x02, Connector_Molex:Molex_PicoBlade_53047-0210_1x02_P1.25mm_Vertical, F.Cu at (85.3, 265.7)
- added REF**: MountingHole_5.5mm, MountingHole:MountingHole_5.5mm, F.Cu at (76.0, 337.2)
- added REF**: MountingHole_5.5mm, MountingHole:MountingHole_5.5mm, F.Cu at (76.3, 255.9)
- added REF**: MountingHole_5.5mm, MountingHole:MountingHole_5.5mm, F.Cu at (76.0, 296.6)
- added REF**: MountingHole_5.5mm, MountingHole:MountingHole_5.5mm, F.Cu at (76.3, 93.3)
- added REF**: MountingHole_5.5mm, MountingHole:MountingHole_5.5mm, F.Cu at (76.0, 133.9)
- added REF**: MountingHole_5.5mm, MountingHole:MountingHole_5.5mm, F.Cu at (76.0, 174.6)
- added REF**: MountingHole_5.5mm, MountingHole:MountingHole_5.5mm, F.Cu at (76.3, 215.3)
- H1: footprint MountingHole:MountingHole_5.5mm_Pad_TopBottom -> MountingHole:MountingHole_5.5mm_Pad
- moved H1 35.6 mm to (76.0, 52.6)
- moved F1 32.4 mm to (95.0, 52.2), turned to -90 degrees
- moved J1 27.6 mm to (85.6, 62.6), turned to 180 degrees
Routing:
- net Net-(F8-Pad1): track 0.00 -> 29.6 mm
- net Net-(F2-Pad1): track 0.00 -> 29.3 mm
- net Net-(F3-Pad1): track 0.00 -> 29.1 mm
- net Net-(F6-Pad1): track 0.00 -> 29.0 mm
- net Net-(F5-Pad1): track 0.00 -> 29.0 mm
- net Net-(F4-Pad1): track 0.00 -> 28.9 mm
- net Net-(F7-Pad1): track 0.00 -> 28.9 mm
- net Net-(F1-Pad1): track 13.5 -> 29.8 mm
- net Net-(J2-Pin_1): track 0.00 -> 11.6 mm
- net Net-(J8-Pin_1): track 0.00 -> 11.4 mm
- net Net-(J7-Pin_1): track 0.00 -> 11.2 mm
- net Net-(J4-Pin_1): track 0.00 -> 11.1 mm
- net Net-(J6-Pin_1): track 0.00 -> 11.0 mm
- net Net-(J5-Pin_1): track 0.00 -> 10.7 mm
- net Net-(J3-Pin_1): track 0.00 -> 9.55 mm
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Other:
- board size 30 x 16 mm -> 30 x 304.9 mm
