File: (LVE)Shutdown_KR/(LVE)Shutdown.kicad_sch (KiCad schematic)
At the start: 109 parts, among them J1 Conn_01x03_Pin, J10 Conn_BTN_Left, J11 Conn_BTN_Right, J12 Conn_BOTS_1, J13 Conn_BOTS_2, J14 Conn_Inertia, J15 Conn_HVD_INTL, J16 Conn_ACC_INTL, J17 Conn_TSMS, J18 Conn_discharge, J19 Conn_precharge, J2 Conn_01x06, J20 Conn_Power, J21 Conn_AIR 1, J22 Conn_AIR 2, J23 Conn_TSAL_OK, J24 IMD_LED, J27 AMS_LED, J3 Conn_01x06, J4 Conn_01x03, J5 IMD_RST, J6 AMS_RST, J8 Conn_BSPD, J9 Conn_BTN_Cockpit, K6 G5Q1A4DC12, K7 G5Q1A4DC12, Q1 2N7000, Q2 2N7000, Q3 2N7000, Q4 2N7000, U1 LM7805MPX/NOPB, U2 SN74AHC1G02DBVR, U6 MC74HC74ADG

Commit message: Slave with SMD and no other fuses
Parts:
- removed Q1, Q2, Q3, Q4: 2N7000, Package_TO_SOT_THT:TO-92_Inline, symbol Transistor_FET:2N7000
- added J7: HV_SENSE_INTL, Connector_JST:JST_XH_B2B-XH-A_1x02_P2.50mm_Vertical, symbol Connector_Generic:Conn_01x02
- added LED15: LTL-1CHG, Kicad_Libraries:LTL1CHG, symbol LTL-1CHG:LTL-1CHG
- added Q1, Q2, Q3, Q5: 2N7002, Package_TO_SOT_SMD:SOT-23, symbol Transistor_FET:2N7002
- added R28, R41: 10k, Resistor_THT:R_Axial_DIN0207_L6.3mm_D2.5mm_P10.16mm_Horizontal, symbol Device:R_Small
- added R29: 27k, Resistor_THT:R_Axial_DIN0207_L6.3mm_D2.5mm_P10.16mm_Horizontal, symbol Device:R_Small
- C1: footprint FA14_Capacitor:FA14X7R1H224KNU00 -> Kicad_Libraries:FA14X7R1H224KNU00
- C2, C6, C7: footprint FA14_Capacitor:FA18X7R1H104KNU00 -> Kicad_Libraries:FA18X7R1H104KNU00
- LED1, LED10, LED11, LED12, LED13, LED14, LED2, LED3, LED4, LED5, LED6, LED7, LED8, LED9: footprint LTL1CHG:LTL1CHG -> Kicad_Libraries:LTL1CHG
Connections:
- net AMS_IN is gone; now on net A: K6.2, K7.3, R3.2, R60.2
- net A: no longer J8.2 (Pin_2), K6.3, R2.2, R59.2
- net AMS_LED-: now also Q3.3 (D)
- net Discharge enable: now also J1.1 (Pin_1); no longer J1.2 (Pin_2)
- net GND: now also J18.1 (Pin_1), LED15.2 (K), Q1.2 (S), Q2.2 (S), Q3.2 (S), Q5.2 (S), R41.2; no longer J18.2 (Pin_2), J4.1 (Pin_1)
- net IMD_LED-: now also Q2.3 (D)
- net Multi purpose enable: now also J1.2 (Pin_2); no longer J1.1 (Pin_1)
- net at R14.1: now also Q2.1 (G)
- net at R2.1, R5.1: now also J4.2 (Pin_2); no longer J4.3 (Pin_3)
- net at R22.1, R36.1: now also J3.1 (Pin_1); no longer J3.2 (Pin_2)
- net at R53.1, R54.1: now also J3.5 (Pin_5); no longer J3.6 (Pin_6)
- net at J17.1 (Pin_1), J22.2 (Pin_2), R52.2: now also J18.2 (Pin_2), J19.2 (Pin_2), R29.2; no longer J18.1 (Pin_1), J19.1 (Pin_1), R53.2
- net at R56.1: now also Q5.1 (G)
- net at D20.2 (A), K6.5: now also Q5.3 (D)
- net at R3.1, R6.1: now also J4.3 (Pin_3); no longer J2.1 (Pin_1)
- net at R16.1, R30.1: now also J2.1 (Pin_1); no longer J2.2 (Pin_2)
- net at R17.1, R31.1: now also J2.2 (Pin_2); no longer J2.3 (Pin_3)
- net at R18.1, R32.1: now also J2.3 (Pin_3); no longer J2.4 (Pin_4)
- net at R19.1, R33.1: now also J2.4 (Pin_4); no longer J2.5 (Pin_5)
- net at R20.1, R34.1: now also J2.5 (Pin_5); no longer J2.6 (Pin_6)
- net at R21.1, R35.1: now also J2.6 (Pin_6); no longer J3.1 (Pin_1)
- net at R23.1, R37.1: now also J3.2 (Pin_2); no longer J3.3 (Pin_3)
- net at R24.1, R38.1: now also J3.3 (Pin_3); no longer J3.4 (Pin_4)
- net at R25.1, R39.1: now also J3.4 (Pin_4); no longer J3.5 (Pin_5)
- net at J21.2 (Pin_2): now also J19.1 (Pin_1); no longer J19.2 (Pin_2)
- net at J17.2 (Pin_2), J23.1 (Pin_1), R50.2: now also R53.2; no longer R25.2
- net at R58.1: now also Q1.1 (G)
- net at D21.2 (A), K7.5: now also Q1.3 (D)
- net at R1.1, R4.1: now also J4.1 (Pin_1); no longer J4.2 (Pin_2)
- net at R24.2, R49.2: now also J16.1 (Pin_1), J7.2 (Pin_2); no longer J16.2 (Pin_2), J23.2 (Pin_2)
- net at J15.1 (Pin_1), R23.2, R48.2: now also J16.2 (Pin_2); no longer J16.1 (Pin_1)
- net at R26.1: now also Q3.1 (G)
- net COCKPIT_IN renamed B
- new net: J3.6 (Pin_6), R29.1, R41.1
- new net: LED15.1 (A), R28.1
- new net: J23.2 (Pin_2), J7.1 (Pin_1), R25.2, R28.2
- new net IMD_IN: J8.2 (Pin_2), K6.3, R2.2, R59.2
Other:
- note added: "1 Shutdown powered 2 BSPD closed 3 IMD closed 4 AMS closed 5 Cockpit closed 6 Left side closed 7 Right Side Closed 8 Brake Over-Travel Switch 1 9 Brake Over-Travel Switch 2 10 Inertia Switch 11 High Voltage Disconnect Interlock 12 Accumulator Connector Interlock 13 HV Sense Interlock 14 TSAL OK 15 Tractive System Master Switch"
- note added: "AIR 2"
- note added: "Discharge Relay"
- note added: "Discharge and multipurpose enable come from BMS master OK_HS comes from IMD"
- note added: "HV Sense Interlock"
- note added: "Pink is the main Shutdown Daisy Chain"
- note added: "Precharge to AIR1"
- note removed: "2 Shutdown powered 3 BSPD closed 4 IMD closed 5 AMS closed 6 Cockpit closed 7 Left side closed 8 Right Side Closed 9 Brake Over-Travel Switch 1 10 Brake Over-Travel Switch 2 11 Inertia Switch 12 High Voltage Disconnect Interlock 13 Accumulator Connector Interlock 14 TSAL OK 15 Tractive System Master Switch"
- note removed: "BSPD LED"
- note removed: "Discharge enable"
- note removed: "Multi purpose enable"
- note removed: "Relays"
- note removed: "Shutdown Circuit"
- note removed: "Shutdown Inputs"
- note removed: "Shutdown Outputs"
- note removed: "Status Monitoring"
- moved on the sheet: C1, C2, C6, C7, J1, J10, J11, J12, J13, J14, J15, J16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

Commit message: added author
Other:
- company: (none) -> UCD Formula Student
Changed lines of the file:
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@@
 	(paper "A2")
 	(title_block
+		(company "UCD Formula Student")
 		(comment 1 "Author: Keelan Reilly")
 	)
