File: ENNOID_BMS/Cell Tap Fuse Board 2x/Cell Tap Fuse Board 2x.kicad_sch (KiCad schematic)
At the start: 3 parts, among them J5 Conn_01x02

Commit message: added author
Other:
- company: (none) -> UCD Formula Student
Changed lines of the file:
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@@
 	(generator_version "9.0")
 	(paper "A4")
+	(title_block
+		(company "UCD Formula Student")
+		(comment 1 "Author: Keelan Reilly")
+	)
 	(no_connect
 		(at 101.6 148.59)
