File: ENNOID_BMS/Cell Tap Fuse Board 3x/Cell Tap Fuse Board 3x.kicad_sch (KiCad schematic)
At the start: 6 parts, among them J1 Conn_01x02, J3 Conn_01x02

Commit message: added author
Other:
- company: (none) -> UCD Formula Student
Changed lines of the file:
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@@
 	(generator_version "9.0")
 	(paper "A4")
+	(title_block
+		(company "UCD Formula Student")
+		(comment 1 "Author: Keelan Reilly")
+	)
 	(no_connect
 		(at 101.6 92.71)
