File: PDU_KR/PDU_KR.kicad_sch (KiCad schematic)
At the start: 44 parts, among them J1 Conn_Supply_A, J10 Conn_Supply_J, J12 Conn_01x02, J2 Conn_Supply_B, J3 Conn_Supply_C, J4 Conn_Supply_D, J5 Conn_Supply_E, J6 Conn_Supply_F, J7 Conn_Supply_G, J8 Conn_Supply_H, J9 Conn_Supply_I

Commit message: added author
Other:
- company: (none) -> UCD Formula Student
Changed lines of the file:
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@@
 	(paper "A3")
 	(title_block
+		(company "UCD Formula Student")
 		(comment 1 "Author: Keelan Reilly")
 	)
