File: ENNOID_BMS/Wiring/MCU.kicad_sch (KiCad schematic)
At the start: 34 parts, among them J15 DEBUG, Q5 BSS138, U12 STM32F303CCTx, U13 LTC6820, U14 LTC6820, Y1 8MHz

Commit message: updated comments
Connections:
- net MA_CELL renamed MA_CELL_P
- net MA_TEMP renamed MA_TEMP_P
- net PA_CELL renamed PA_CELL_N
- net PA_TEMP renamed PA_TEMP_N
