File: Kieran Care package/BSPD_KR/BSPD KiCAD.kicad_sch (KiCad schematic)
At the start: 65 parts, among them J1 Conn_01x03, J2 Conn_01x02, J3 Conn_01x02, K1 G5Q-1A4-DC12, Q1 2N7002, Q3 2N7002, U18 SN74AHCT1G08DBVR, U19 LM339N, U4 LM7805MPX/NOPB, U5 LM339N, U6 SN74AHC1G02DBVR, U9 SN74LVC1G04DBVT

Commit message: updated comments
Other:
- note removed: "ALl LEDs are off when BSPD is OK"
- note removed: "Anything below 0.455 volts is invalid 20 bar corresponds 2.8V 25 bar corresponds to 3.36V 30 bar correspons to 3.93v"
- note removed: "BSPD is closed when NOT( hard braking AND too much power for >500 ms )"
- note removed: "LED5 OFF = relay closed LED5 ON = relay open"
- note removed: "Should be set to whatever sensor outputs at 16A V_threshold = 2.5 V + (15.9 A × 0.010 V/A) ≈ 2.66 V or better: TP4 = zero-current sensor voltage + 0.16 V"
Changed lines of the file:
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@@
 		(comment 2 "Updated by: Keelan Reilly")
-	)
-	(text "Should be set to whatever sensor outputs at 16A\n\nV_threshold = 2.5 V + (15.9 A × 0.010 V/A) ≈ 2.66 V\n\nor better:\n\nTP4 = zero-current sensor voltage + 0.16 V\n\n"
-		(exclude_from_sim no)
-		(at 89.916 87.122 0)
-		(effects
-			(font
-				(size 1.27 1.27)
-			)
-		)
 	)
 	(text "NOR Logic"
@@
 		)
 	)
-	(text "ALl LEDs are off when BSPD is OK"
-		(exclude_from_sim no)
-		(at 85.598 172.466 0)
-		(effects
-			(font
-				(size 1.27 1.27)
-			)
-		)
-	)
 	(text "Orion BMS Current Sesor"
 		(exclude_from_sim no)
@@
 		)
 	)
-	(text "Anything below 0.455 volts is invalid\n20 bar corresponds 2.8V\n25 bar corresponds to 3.36V\n30 bar correspons to 3.93v"
-		(exclude_from_sim no)
-		(at 96.266 136.906 0)
-		(effects
-			(font
-				(size 1.27 1.27)
-			)
-		)
-	)
 	(text "Brake Pressure Sensor FRONT"
 		(exclude_from_sim no)
@@
 		)
 	)
-	(text "BSPD is closed when NOT( hard braking AND too much power for >500 ms )"
-		(exclude_from_sim no)
-		(at 79.756 106.172 0)
-		(effects
-			(font
-				(size 1.27 1.27)
-			)
-		)
-	)
 	(text "Brake Pressure Sensor REAR"
 		(exclude_from_sim no)
@@
 		)
 	)
-	(text "LED5 OFF = relay closed\n\nLED5 ON  = relay open"
-		(exclude_from_sim no)
-		(at 366.268 93.472 0)
-		(effects
-			(font
-				(size 1.27 1.27)
-			)
-		)
-	)
 	(junction
 		(at 137.16 46.99)
@@
 	)
 	(junction
-		(at 290.83 129.54)
-		(diameter 0)
-		(color 0 0 0 0)
-	)
-	(junction
 		(at 160.02 86.36)
 		(diameter 1.016)
@@
 	(wire
 		(pts
+			(xy 289.56 129.54) (xy 300.99 129.54)
+		)
+		(stroke
+			(width 0)
+			(type solid)
+		)
+	)
+	(wire
+		(pts
 			(xy 170.18 97.79) (xy 171.45 97.79)
 		)
@@
 	(wire
 		(pts
-			(xy 290.83 129.54) (xy 300.99 129.54)
-		)
-		(stroke
-			(width 0)
-			(type solid)
-		)
-	)
-	(wire
-		(pts
 			(xy 195.58 120.65) (xy 198.12 120.65)
 		)
@@
 		(pts
 			(xy 312.42 93.98) (xy 312.42 106.68)
-		)
-		(stroke
-			(width 0)
-			(type default)
-		)
-	)
-	(wire
-		(pts
-			(xy 290.83 129.54) (xy 289.56 129.54)
 		)
 		(stroke
@@
 	(wire
 		(pts
-			(xy 290.83 128.27) (xy 290.83 129.54)
-		)
-		(stroke
-			(width 0)
-			(type default)
-		)
-	)
-	(wire
-		(pts
 			(xy 175.26 72.39) (xy 175.26 73.66)
 		)
@@
 	)
 	(label "10s"
-		(at 290.83 128.27 0)
+		(at 289.56 129.54 0)
 		(effects
 			(font
