File: Kieran Care package/Charger_Shutdown_KR/Charger_Shutdown_KR.kicad_sch (KiCad schematic)
At the start: 43 parts, among them J1 Conn_01x02_Pin, J2 Conn_01x02_Pin, J3 Conn_01x04_Pin, J4 Conn_01x02_Pin, J5 Conn_01x02_Pin, J6 Conn_01x02_Pin, J7 Conn_01x04_Pin, J8 Conn_01x04_Pin, J9 Conn_01x02_Pin, K1 G5Q1A4DC12, Q1 2N7000, Q2 2N7000, Q3 2N7000, SW1 SW_SPST, SW2 SW_SPST, U1 SN74AHC1G04DBVRE4, U2 SN74LS21DR, U3 MC74HC74ADG, U5 LM7805MPX/NOPB, U6 SN74AHC1G02DBVR

Commit message: updated comments
Parts:
- removed SW1, SW2: SW_SPST, symbol Switch:SW_SPST
Other:
- note removed: "HVIl1"
- note removed: "HVIl2"
- note removed: "This is redundant Precharge relay is not a part of charger path (probably...)"
Changed lines of the file:
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@@
 		(comment 1 "Author: Keelan Reilly")
 	)
-	(text "HVIl1"
-		(exclude_from_sim no)
-		(at -40.386 71.882 0)
-		(effects
-			(font
-				(size 1.27 1.27)
-			)
-		)
-	)
 	(text "test commit 1"
 		(exclude_from_sim no)
@@
 		)
 	)
-	(text "This is redundant\nPrecharge relay is not a part of charger path\n(probably...)"
-		(exclude_from_sim no)
-		(at 37.338 189.484 0)
-		(effects
-			(font
-				(size 1.27 1.27)
-			)
-		)
-	)
 	(text "Manual Reset Button"
 		(exclude_from_sim no)
@@
 		)
 	)
-	(text "HVIl2"
-		(exclude_from_sim no)
-		(at -22.098 71.882 0)
-		(effects
-			(font
-				(size 1.27 1.27)
-			)
-		)
-	)
 	(text "IMD NOT OK latches LOW, making Q' HIGH"
 		(exclude_from_sim no)
@@
 	(wire
 		(pts
-			(xy -55.88 83.82) (xy -44.45 83.82)
-		)
-		(stroke
-			(width 0)
-			(type default)
-		)
-	)
-	(wire
-		(pts
 			(xy 251.46 135.89) (xy 248.92 135.89)
 		)
@@
 	(wire
 		(pts
-			(xy -16.51 83.82) (xy -6.35 83.82)
-		)
-		(stroke
-			(width 0)
-			(type default)
-		)
-	)
-	(wire
-		(pts
 			(xy 66.04 58.42) (xy 66.04 62.23)
 		)
@@
 	(wire
 		(pts
-			(xy -34.29 83.82) (xy -26.67 83.82)
-		)
-		(stroke
-			(width 0)
-			(type default)
-		)
-	)
-	(wire
-		(pts
 			(xy 143.51 195.58) (xy 147.32 195.58)
 		)
@@
 		)
 	)
-	(global_label "HVIL-"
-		(shape input)
-		(at -6.35 83.82 0)
-		(fields_autoplaced yes)
-		(effects
-			(font
-				(size 1.27 1.27)
-			)
-			(justify left)
-		)
-		(property "Intersheetrefs" "${INTERSHEET_REFS}"
-			(at 2.2596 83.82 0)
-			(effects
-				(font
-					(size 1.27 1.27)
-				)
-				(justify left)
-				(hide yes)
-			)
-		)
-	)
 	(global_label "AIR1_open"
 		(shape input)
@@
 		)
 	)
-	(global_label "Charger_12V+"
-		(shape input)
-		(at -55.88 83.82 180)
-		(fields_autoplaced yes)
-		(effects
-			(font
-				(size 1.27 1.27)
-			)
-			(justify right)
-		)
-		(property "Intersheetrefs" "${INTERSHEET_REFS}"
-			(at -72.2908 83.82 0)
-			(effects
-				(font
-					(size 1.27 1.27)
-				)
-				(justify right)
-				(hide yes)
-			)
-		)
-	)
 	(global_label "SAFE_LED-"
 		(shape input)
@@
 	)
 	(symbol
-		(lib_id "Switch:SW_SPST")
-		(at -39.37 83.82 0)
-		(unit 1)
-		(exclude_from_sim no)
-		(in_bom yes)
-		(on_board yes)
-		(dnp no)
-		(fields_autoplaced yes)
-		(property "Reference" "SW1"
-			(at -39.37 77.47 0)
-			(effects
-				(font
-					(size 1.27 1.27)
-				)
-			)
-		)
-		(property "Value" "SW_SPST"
-			(at -39.37 80.01 0)
-			(effects
-				(font
-					(size 1.27 1.27)
-				)
-			)
-		)
-		(property "Footprint" ""
-			(at -39.37 83.82 0)
-			(effects
-				(font
-					(size 1.27 1.27)
-				)
-				(hide yes)
-			)
-		)
-		(property "Datasheet" "~"
-			(at -39.37 83.82 0)
-			(effects
-				(font
-					(size 1.27 1.27)
-				)
-				(hide yes)
-			)
-		)
-		(property "Description" "Single Pole Single Throw (SPST) switch"
-			(at -39.37 83.82 0)
-			(effects
-				(font
-					(size 1.27 1.27)
-				)
-				(hide yes)
-			)
-		)
-		(pin "2"
-		)
-		(pin "1"
-		)
-		(instances
-			(project ""
-				(path "/ba2fd4c7-be96-4612-905b-530e6de824dd"
-					(reference "SW1")
-					(unit 1)
-				)
-			)
-		)
-	)
-	(symbol
 		(lib_id "74xx:74HC74")
 		(at 289.56 132.08 90)
@@
 					(unit 1)
 				)
-			)
-		)
-	)
-	(symbol
-		(lib_id "Switch:SW_SPST")
-		(at -21.59 83.82 0)
-		(unit 1)
-		(exclude_from_sim no)
-		(in_bom yes)
-		(on_board yes)
-		(dnp no)
-		(fields_autoplaced yes)
-		(property "Reference" "SW2"
-			(at -21.59 77.47 0)
-			(effects
-				(font
-					(size 1.27 1.27)
-				)
-			)
-		)
-		(property "Value" "SW_SPST"
-			(at -21.59 80.01 0)
-			(effects
-				(font
-					(size 1.27 1.27)
-				)
-			)
-		)
-		(property "Footprint" ""
-			(at -21.59 83.82 0)
-			(effects
-				(font
-					(size 1.27 1.27)
-				)
-				(hide yes)
-			)
-		)
-		(property "Datasheet" "~"
-			(at -21.59 83.82 0)
-			(effects
-				(font
-					(size 1.27 1.27)
-				)
-				(hide yes)
-			)
-		)
-		(property "Description" "Single Pole Single Throw (SPST) switch"
-			(at -21.59 83.82 0)
-			(effects
-				(font
-					(size 1.27 1.27)
-				)
-				(hide yes)
-			)
-		)
-		(pin "2"
-		)
-		(pin "1"
-		)
-		(instances
-			(project "Charger_Shutdown_KR"
-				(path "/ba2fd4c7-be96-4612-905b-530e6de824dd"
-					(reference "SW2")
-					(unit 1)
-				)
