File: Kieran Care package/ENNOID_BMS - Master/MCU.kicad_sch (KiCad schematic)
At the start: 34 parts, among them J15 DEBUG, Q5 BSS138, U12 STM32F303CCTx, U13 LTC6820, U14 LTC6820, Y1 8MHz

Commit message: updated comments
Changed lines of the file:
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@@
 	)
 	(hierarchical_label "MA_CELL"
-		(shape output)
+		(shape input)
 		(at 317.5 48.26 180)
 		(effects
@@
 	)
 	(hierarchical_label "PA_TEMP"
-		(shape output)
+		(shape input)
 		(at 318.77 128.27 180)
 		(effects
@@
 	)
 	(hierarchical_label "MA_TEMP"
-		(shape output)
+		(shape input)
 		(at 318.77 118.11 180)
 		(effects
@@
 	)
 	(hierarchical_label "PA_CELL"
-		(shape output)
+		(shape input)
 		(at 317.5 58.42 180)
 		(effects
