File: Kieran Care package/ENNOID_BMS - Master/PowerSupply.kicad_sch (KiCad schematic)
At the start: 33 parts, among them J14 Charger, Q1 BSS138, Q2 BSS138, Q3 BSS138, Q4 BSS138, U11 LM5165YDRC

Commit message: updated comments
Other:
- note removed: "If USB or CAN is connected enable request goes low They are an external wake request for MCU"
Changed lines of the file:
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@@
-		)
-	)
-	(text "If USB or CAN is connected enable request goes low\nThey are an external wake request for MCU"
-		(exclude_from_sim no)
-		(at 425.958 219.456 0)
-		(effects
-			(font
-				(size 1.27 1.27)
-			)
 		)
 	)
