File: Kieran Care package/NEW_TSAL_KR/TSAL.kicad_sch (KiCad schematic)
At the start: 99 parts, among them IC1 CD4072BE, IC3 SN74HC86N, IC4 CD4072BE, IC5 CD4072BE, J1 B4B-XH-A, J2 B3B-XH-A, J3 B2B-XH-A, J4 B4B-XH-A, J5 B4B-XH-A, J6 B2B-XH-A, J7 B2B-XH-A, J8 B2B-XH-A, K1 G5RL-K1-E-DC5, K2 G5Q1A4DC12, Q1 2N7000, Q2 2N7000, Q3 2N7000, Q4 2N7000, Q5 2N7000, Q6 2N7000, Q7 2N7000, U1 SN74AHC1G32TDBVRQ1, U14 SN74AHCT1G08DBVR, U2 LMC555CMX/NOPB, U26 LM2596SX-5.0/NOPB, U3 LM339N/NOPB, U4 LM339N/NOPB, U5 LM339N/NOPB, U6 LMC555CMX/NOPB, U7 SN74AHC1G32TDBVRQ1, U8 SN74AHCT1G08DBVR, U9 SN74AHC1G04DBVRE4

Commit message: updated comments
Other:
- note removed: "This is wrong, these are both digital signals, High or Low. The precharge Relay is not like the AIRS"
Changed lines of the file:
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@@
-		)
-	)
-	(text "This is wrong, these are both digital signals, High or Low.\nThe precharge Relay is not like the AIRS"
-		(exclude_from_sim no)
-		(at 256.54 292.862 0)
-		(effects
-			(font
-				(size 1.27 1.27)
-			)
 		)
 	)
