File: Kieran Care package/Teensy 4.1 Breakout Board/Breakout.kicad_sch (KiCad schematic)
At the start: 55 parts, among them J1 CAN, J10 RTD_Speaker, J11 Current Sensor Power source, J12 RTD_button, J2 12V Power, J3 APPS1, J4 APPS2, J5 Brake_Pressure_Front, J6 Brake_Pressure_Rear, J7 Nextion, J8 ESP32, J9 Brake_Light, Q1 2N7002, Q3 2N7002, U1 SN65HVD230, U3 Teensy4.1, U4 TPS62163DSG, U5 MPU6050

Commit message: updated comments
Parts:
- removed C11: 0.1uF, FA14_Capacitor:FA18X7R1H104KNU00, symbol Device:C
- removed R21: 220, Resistor_THT:R_Axial_DIN0207_L6.3mm_D2.5mm_P10.16mm_Horizontal, symbol Device:R
